Commit message: Added new frames l_end_eff and r_end_eff after l_palm and r_palm for manipulation purpose.

File: urdf/atlas_v5_robotiq.urdf (robot description, URDF)
Before this commit: robot atlas, 127 links, 126 joints
Links:
- added link l_end_eff
- added link r_end_eff
Joints:
- added joint l_robotiq_end_eff_virtual_joint: type fixed, parent l_palm, child l_end_eff, origin xyz=0.0 0.1 0.0 rpy=0 0 1.5708
- added joint r_robotiq_end_eff_virtual_joint: type fixed, parent r_palm, child r_end_eff, origin xyz=0.0 0.1 0.0 rpy=3.14159265 0.0 1.57079633
