Commit message: added dummy end effector frames for taskspace planning

File: urdf/atlas_unplugged_v5_no_hands.urdf (robot description, URDF)
Before this commit: robot atlas, 47 links, 46 joints
Links:
- added link l_end_eff
- added link l_palm
- added link r_end_eff
- added link r_palm
Joints:
- added joint l_robotiq_end_eff_virtual_joint: type fixed, parent l_palm, child l_end_eff, origin xyz=0.0 0.1 0.0 rpy=0 0 1.5708
- added joint l_robotiq_hand_joint: type fixed, parent l_hand, child l_palm, origin xyz=-0.00125 0.17 0.01 rpy=3.14159 3.14159 3.14159
- added joint r_robotiq_end_eff_virtual_joint: type fixed, parent r_palm, child r_end_eff, origin xyz=0.0 0.1 0.0 rpy=3.14159265 0.0 1.57079633
- added joint r_robotiq_hand_joint: type fixed, parent r_hand, child r_palm, origin xyz=-0.00125 -0.17 0.01 rpy=3.14159 0 0
